File: Knox Key Kicad.kicad_pcb (KiCad board)
At the start: 2 copper layers, 27.2 x 17.1 mm, 29 parts, among them J1 Conn_01x04_Pin, P1 USB_C_Plug_USB2.0, SW1 SW_Push, U2 ATECC608B-MAHDA, U3 MCP1700x-330xxTT, U4 USBLC6-2SC6, U6 STM32L431CBTx, Y1 8MHz

Commit message: Update
Parts:
- removed J1: Conn_01x04_Pin, Connector_PinHeader_2.54mm:PinHeader_1x04_P2.54mm_Vertical
- added J3: Conn_01x05, Connector_PinHeader_2.54mm:PinHeader_1x05_P2.54mm_Vertical, F.Cu at (157.9, 102.0)
- moved R6 0.41 mm to (155.9, 111.2)
- moved R7 0.41 mm to (155.9, 113.2)
- moved R8 0.41 mm to (155.9, 115.1)
Connections:
- C7 pad 1: GND -> /BOOT0
Routing:
- net /NRST: track 6.32 -> 28.6 mm, vias 0 -> 1
- net GND: track 22.1 -> 30.1 mm, vias 27 -> 25
- net +3V3: track 82.5 -> 76.3 mm
- net /BOOT0: track 4.33 -> 7.35 mm, vias 0 -> 2
- net /SWCLK: track 12.0 -> 9.60 mm
- net /SWDIO: track 10.1 -> 9.37 mm
- net Net-(D1-GK): track 8.08 -> 8.01 mm, vias 0 -> 2
- removed copper zone on F.Cu, net GND
Other:
- board text added: "GND NRST SWCLK SWDIO +3V3"
- board text removed: "GND SWCLK SWDIO +3V3"
