File: Knox Key Kicad.kicad_sch (KiCad schematic)
At the start: 29 parts, among them J1 Conn_01x04_Pin, SW1 SW_Push, U2 ATECC608B-MAHDA, U3 MCP1700x-330xxTT, U4 USBLC6-2SC6, U6 STM32L431CBTx, Y1 8MHz

Commit message: Update
Parts:
- removed J1: Conn_01x04_Pin, Connector_PinHeader_2.54mm:PinHeader_1x04_P2.54mm_Vertical, symbol Connector:Conn_01x04_Pin
- added J3: Conn_01x05, Connector_PinHeader_2.54mm:PinHeader_1x05_P2.54mm_Vertical, symbol Connector_Generic:Conn_01x05
- R1: value 10k -> 5.1k; Distributer Link https://www.lcsc.com/product-detail/Chip-Resistor-Surface-Mount_YAGEO-RC0402FR-0710KL_C60490.html -> https://www.lcsc.com/product-detail/Chip-Resistor-Surface-Mount_UNI-ROYAL-Uniroyal-Elec-0402WGJ0472TCE_C25940.html; LCSC C60490 -> C25940; Manufacturer YAGEO -> UNI-ROYAL(Uniroyal Elec); Manufacturer Part Number RC0402FR-0710KL -> 0402WGJ0472TCE
- R4: value 4k7 -> 5.1k
Connections:
- net +3V3: now also D1.4 (A), J3.1 (Pin_1)
- net BOOT0: now also C7.1; no longer R1.2
- net GND: now also J3.5 (Pin_5); no longer C7.1, D1.4 (A)
- net NRST: now also J3.4 (Pin_4)
- net SWCLK: now also J3.3 (Pin_3)
- net SWDIO: now also J3.2 (Pin_2)
- net USB_CONN_D+: now also USB1.B6 (D+)
- net USB_CONN_D-: now also USB1.B7 (D-)
- net at R8.1: now also D1.3 (BK); no longer D1.1 (RK)
- net at R6.1: now also D1.1 (RK); no longer D1.3 (BK)
- net at USB1.B5 (CC2): now also R1.2
- no-connect marks 38 -> 35
